File: pcb/Keyboard-2600/Keyboard-2600.kicad_sch (KiCad schematic)
At the start: 28 parts, among them J1 USB_A, J2 Left Forward Port, J3 Right Forward Port, J4 2600 Joystick Connector, J5 Mini-DIN-6, J6 Expansion Port, SW1 Config Switch-Box, SW2 Reset, U1 ATmega328P-A, U2 74HC4066D_653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

Commit message: Test board WIP state.
Parts:
- removed J4: 2600 Joystick Connector, Connector_PinHeader_2.54mm:PinHeader_2x09_P2.54mm_Vertical, symbol Connector_Generic:Conn_02x09_Odd_Even
- removed J6: Expansion Port, Connector_PinHeader_2.54mm:PinHeader_2x13_P2.54mm_Vertical, symbol Connector_Generic:Conn_02x13_Odd_Even
- added J6: Expansion Port, KeyPortari:PinHeader_2x14_P2.54mm_Vertical_KeyPortari_Expansion-Port, symbol Connector_Generic:Conn_02x14_Odd_Even
- added J7: Joystick right, Connector_PinHeader_2.54mm:PinHeader_2x05_P2.54mm_Vertical, symbol Connector_Generic:Conn_02x05_Top_Bottom
- added J8: Joystick left, Connector_PinHeader_2.54mm:PinHeader_2x05_P2.54mm_Vertical, symbol Connector_Generic:Conn_02x05_Top_Bottom
- J5: footprint 2600-Keyboard:Connector_Mini-DIN_Female_6Pin_2rows -> KeyPortari:Connector_Mini-DIN_Female_6Pin_2rows
- R5, R6: footprint Resistor_SMD:R_0402_1005Metric -> Resistor_SMD:R_0603_1608Metric
- U2, U3: footprint 74HC4066D_653f:SOIC127P600X175-14N -> Package_SO:SOIC-14_3.9x8.7mm_P1.27mm
Connections:
- net +5V: now also J6.2 (Pin_2), J7.7 (Pin_7), J8.7 (Pin_7)
- net A0: now also J6.4 (Pin_4); no longer R2.1, R3.1, R4.1, R5.1, R6.1
- net A1: now also J6.6 (Pin_6)
- net A2: now also J6.8 (Pin_8)
- net A3: now also J6.10 (Pin_10)
- net A4: now also J6.20 (Pin_20)
- net A5: now also J6.22 (Pin_22)
- net A7: now also J6.28 (Pin_28)
- net CLK: now also U1.13 (PB1); no longer U1.12 (PB0)
- net DATA: now also U1.12 (PB0); no longer U1.13 (PB1)
- net GND: now also J6.1 (Pin_1), J7.8 (Pin_8), J8.8 (Pin_8)
- net I0: now also J6.3 (Pin_3), J8.5 (Pin_5)
- net I1: now also J6.5 (Pin_5), J8.9 (Pin_9)
- net I2: now also J6.7 (Pin_7), J7.5 (Pin_5)
- net I3: now also J6.9 (Pin_9), J7.9 (Pin_9)
- net I4: now also J6.24 (Pin_24), J8.6 (Pin_6)
- net I5: now also J6.26 (Pin_26), J7.6 (Pin_6)
- net OE_L: now also J6.21 (Pin_21)
- net OE_R: now also J6.19 (Pin_19)
- net PA0: now also J6.12 (Pin_12), J7.1 (Pin_1)
- net PA1: now also J6.14 (Pin_14), J7.2 (Pin_2)
- net PA2: now also J6.16 (Pin_16), J7.3 (Pin_3)
- net PA3: now also J6.18 (Pin_18), J7.4 (Pin_4)
- net PA4: now also J6.11 (Pin_11), J8.1 (Pin_1)
- net PA5: now also J6.13 (Pin_13), J8.2 (Pin_2)
- net PA6: now also J6.15 (Pin_15), J8.3 (Pin_3)
- net PA7: now also J6.17 (Pin_17), J8.4 (Pin_4)
- net PB2: now also J6.23 (Pin_23)
- net PB3: now also J6.25 (Pin_25)
- net RST: now reaches C3.1, R1.1, SW2.2, U1.29 (~{RESET}/PC6)
- net RST: now also J6.27 (Pin_27)
- net A6 renamed CONF
- net CONF: now also R2.1, R3.1, R4.1, R5.1, R6.1
- no-connect marks 2 -> 4
Other:
- company: (none) -> Wolfgang Stubig
- title: (none) -> KeyPortari
- moved on the sheet: H1, H2, H3, H4, J5, R1
